File: cad/electrical/Motherboard.brd (EAGLE design)
At the start: 130 x 130 mm, 56 parts, among them J1 POWER_JACKPTH_LOCK, J2 FEMALE 2x3, J3 FEMALE 2x3, U1 LM358

Commit message: Imported robot code and electrical CAD
Parts:
- R1, R7: value (none) -> 10k
- R10: value (none) -> 5.6k
- R11: value (none) -> 5k
- R12, R9: value (none) -> 100k
- R2: value (none) -> 270
- R3, R4, R5: value (none) -> 160
- R6: value (none) -> 47k
- R8: value (none) -> 30k
Changed lines of the file:
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@@
 <attribute name="VALUE" x="8.382" y="29.21" size="0.6096" layer="27" font="vector" ratio="20" rot="R90"/>
 </element>
-<element name="R1" library="rcl" library_urn="urn:adsk.eagle:library:334" package="0207/10" package3d_urn="urn:adsk.eagle:package:23491/2" value="" x="-15.24" y="50.8" smashed="yes" rot="R270">
+<element name="R1" library="rcl" library_urn="urn:adsk.eagle:library:334" package="0207/10" package3d_urn="urn:adsk.eagle:package:23491/2" value="10k" x="-15.24" y="50.8" smashed="yes" rot="R270">
 <attribute name="NAME" x="-13.716" y="53.848" size="1.27" layer="25" ratio="10" rot="R270"/>
 <attribute name="SPICEPREFIX" value="R" x="-15.24" y="50.8" size="1.778" layer="27" rot="R270" display="off"/>
 <attribute name="VALUE" x="-15.875" y="53.0606" size="1.27" layer="27" ratio="10" rot="R270"/>
 </element>
-<element name="R2" library="rcl" library_urn="urn:adsk.eagle:library:334" package="0207/10" package3d_urn="urn:adsk.eagle:package:23491/2" value="" x="15.24" y="50.8" smashed="yes" rot="R270">
+<element name="R2" library="rcl" library_urn="urn:adsk.eagle:library:334" package="0207/10" package3d_urn="urn:adsk.eagle:package:23491/2" value="270" x="15.24" y="50.8" smashed="yes" rot="R270">
 <attribute name="NAME" x="16.764" y="53.848" size="1.27" layer="25" ratio="10" rot="R270"/>
 <attribute name="SPICEPREFIX" value="R" x="15.24" y="50.8" size="1.778" layer="27" rot="R270" display="off"/>
 <attribute name="VALUE" x="14.605" y="53.0606" size="1.27" layer="27" ratio="10" rot="R270"/>
 </element>
-<element name="R3" library="rcl" library_urn="urn:adsk.eagle:library:334" package="0207/10" package3d_urn="urn:adsk.eagle:package:23491/2" value="" x="-3.81" y="27.94" smashed="yes">
+<element name="R3" library="rcl" library_urn="urn:adsk.eagle:library:334" package="0207/10" package3d_urn="urn:adsk.eagle:package:23491/2" value="160" x="-3.81" y="27.94" smashed="yes">
 <attribute name="NAME" x="-6.858" y="29.464" size="1.27" layer="25" ratio="10"/>
 <attribute name="SPICEPREFIX" value="R" x="-3.81" y="27.94" size="1.778" layer="27" display="off"/>
 <attribute name="VALUE" x="-6.0706" y="27.305" size="1.27" layer="27" ratio="10"/>
 </element>
-<element name="R4" library="rcl" library_urn="urn:adsk.eagle:library:334" package="0207/10" package3d_urn="urn:adsk.eagle:package:23491/2" value="" x="1.27" y="20.32" smashed="yes">
+<element name="R4" library="rcl" library_urn="urn:adsk.eagle:library:334" package="0207/10" package3d_urn="urn:adsk.eagle:package:23491/2" value="160" x="1.27" y="20.32" smashed="yes">
 <attribute name="NAME" x="-1.778" y="21.844" size="1.27" layer="25" ratio="10"/>
 <attribute name="SPICEPREFIX" value="R" x="1.27" y="20.32" size="1.778" layer="27" display="off"/>
 <attribute name="VALUE" x="-0.9906" y="19.685" size="1.27" layer="27" ratio="10"/>
 </element>
-<element name="R5" library="rcl" library_urn="urn:adsk.eagle:library:334" package="0207/10" package3d_urn="urn:adsk.eagle:package:23491/2" value="" x="1.27" y="16.51" smashed="yes">
+<element name="R5" library="rcl" library_urn="urn:adsk.eagle:library:334" package="0207/10" package3d_urn="urn:adsk.eagle:package:23491/2" value="160" x="1.27" y="16.51" smashed="yes">
 <attribute name="NAME" x="-1.778" y="18.034" size="1.27" layer="25" ratio="10"/>
 <attribute name="SPICEPREFIX" value="R" x="1.27" y="16.51" size="1.778" layer="27" display="off"/>
@@
 <attribute name="VALUE" x="-48.26" y="22.86" size="0.6096" layer="27" font="vector" ratio="20" rot="R180" align="bottom-center"/>
 </element>
-<element name="R6" library="rcl" library_urn="urn:adsk.eagle:library:334" package="0207/10" package3d_urn="urn:adsk.eagle:package:23491/2" value="" x="-46.99" y="24.13" smashed="yes" rot="R180">
+<element name="R6" library="rcl" library_urn="urn:adsk.eagle:library:334" package="0207/10" package3d_urn="urn:adsk.eagle:package:23491/2" value="47k" x="-46.99" y="24.13" smashed="yes" rot="R180">
 <attribute name="NAME" x="-43.942" y="22.606" size="1.27" layer="25" ratio="10" rot="R180"/>
 <attribute name="SPICEPREFIX" value="R" x="-46.99" y="24.13" size="1.778" layer="27" rot="R180" display="off"/>
 <attribute name="VALUE" x="-44.7294" y="24.765" size="1.27" layer="27" ratio="10" rot="R180"/>
 </element>
-<element name="R7" library="rcl" library_urn="urn:adsk.eagle:library:334" package="0207/10" package3d_urn="urn:adsk.eagle:package:23491/2" value="" x="-46.99" y="26.67" smashed="yes">
+<element name="R7" library="rcl" library_urn="urn:adsk.eagle:library:334" package="0207/10" package3d_urn="urn:adsk.eagle:package:23491/2" value="10k" x="-46.99" y="26.67" smashed="yes">
 <attribute name="NAME" x="-50.038" y="28.194" size="1.27" layer="25" ratio="10"/>
 <attribute name="SPICEPREFIX" value="R" x="-46.99" y="26.67" size="1.778" layer="27" display="off"/>
 <attribute name="VALUE" x="-49.2506" y="26.035" size="1.27" layer="27" ratio="10"/>
 </element>
-<element name="R8" library="rcl" library_urn="urn:adsk.eagle:library:334" package="0207/10" package3d_urn="urn:adsk.eagle:package:23491/2" value="" x="-48.26" y="3.81" smashed="yes" rot="R90">
+<element name="R8" library="rcl" library_urn="urn:adsk.eagle:library:334" package="0207/10" package3d_urn="urn:adsk.eagle:package:23491/2" value="30k" x="-48.26" y="3.81" smashed="yes" rot="R90">
 <attribute name="NAME" x="-49.784" y="0.762" size="1.27" layer="25" ratio="10" rot="R90"/>
 <attribute name="SPICEPREFIX" value="R" x="-48.26" y="3.81" size="1.778" layer="27" rot="R90" display="off"/>
 <attribute name="VALUE" x="-47.625" y="1.5494" size="1.27" layer="27" ratio="10" rot="R90"/>
 </element>
-<element name="R10" library="rcl" library_urn="urn:adsk.eagle:library:334" package="0207/10" package3d_urn="urn:adsk.eagle:package:23491/2" value="" x="-29.21" y="26.67" smashed="yes" rot="MR0">
+<element name="R10" library="rcl" library_urn="urn:adsk.eagle:library:334" package="0207/10" package3d_urn="urn:adsk.eagle:package:23491/2" value="5.6k" x="-29.21" y="26.67" smashed="yes" rot="MR0">
 <attribute name="NAME" x="-26.162" y="28.194" size="1.27" layer="26" ratio="10" rot="MR0"/>
 <attribute name="SPICEPREFIX" value="R" x="-29.21" y="26.67" size="1.778" layer="28" rot="MR0" display="off"/>
@@
 <attribute name="VALUE" x="5.08" y="-26.924" size="0.6096" layer="27" font="vector" ratio="20" align="top-left"/>
 </element>
-<element name="R11" library="pot" library_urn="urn:adsk.eagle:library:331" package="B25P" package3d_urn="urn:adsk.eagle:package:22684/1" value="" x="-57.15" y="2.54" smashed="yes" rot="R90">
+<element name="R11" library="pot" library_urn="urn:adsk.eagle:library:331" package="B25P" package3d_urn="urn:adsk.eagle:package:22684/1" value="5k" x="-57.15" y="2.54" smashed="yes" rot="R90">
 <attribute name="NAME" x="-60.96" y="-0.635" size="1.27" layer="25" ratio="10" rot="R90"/>
 <attribute name="VALUE" x="-52.07" y="-0.6096" size="1.27" layer="27" ratio="10" rot="R90"/>
 </element>
-<element name="R9" library="rcl" library_urn="urn:adsk.eagle:library:334" package="0207/10" package3d_urn="urn:adsk.eagle:package:23491/2" value="" x="-54.61" y="13.97" smashed="yes" rot="R90">
+<element name="R9" library="rcl" library_urn="urn:adsk.eagle:library:334" package="0207/10" package3d_urn="urn:adsk.eagle:package:23491/2" value="100k" x="-54.61" y="13.97" smashed="yes" rot="R90">
 <attribute name="NAME" x="-56.134" y="10.922" size="1.27" layer="25" ratio="10" rot="R90"/>
 <attribute name="SPICEPREFIX" value="R" x="-54.61" y="13.97" size="1.778" layer="27" rot="R90" display="off"/>
 <attribute name="VALUE" x="-53.975" y="11.7094" size="1.27" layer="27" ratio="10" rot="R90"/>
 </element>
-<element name="R12" library="rcl" library_urn="urn:adsk.eagle:library:334" package="0207/10" package3d_urn="urn:adsk.eagle:package:23491/2" value="" x="-58.42" y="13.97" smashed="yes" rot="R90">
+<element name="R12" library="rcl" library_urn="urn:adsk.eagle:library:334" package="0207/10" package3d_urn="urn:adsk.eagle:package:23491/2" value="100k" x="-58.42" y="13.97" smashed="yes" rot="R90">
 <attribute name="NAME" x="-59.944" y="10.922" size="1.27" layer="25" ratio="10" rot="R90"/>
 <attribute name="SPICEPREFIX" value="R" x="-58.42" y="13.97" size="1.778" layer="27" rot="R90" display="off"/>
